File: Hardware/Photon Battery Shield.brd (EAGLE design)
At the start: 40.6 x 35.6 mm, 24 parts, among them U1 MAX1704X, U2 MCP73831

Commit message: Fixing board name silk.
Parts:
- moved FID2 2.84 mm to (3.81, 29.2)
- moved D2 2.54 mm to (26.7, 33.0)
- moved C1 2.54 mm to (16.5, 14.0)
- moved D1 2.54 mm to (16.5, 19.1)
- moved LOGO2 2.54 mm to (14.2, 1.78)
- moved R3 2.54 mm to (16.5, 7.62)
- moved U2 2.54 mm to (16.5, 11.4)
- moved JP3 2.54 mm to (10.2, 0.00)
- moved LOGO3 2.54 mm to (5.59, 10.8)
- moved C2 2.54 mm to (24.1, 8.89)
- moved C3 2.54 mm to (19.7, 14.0)
- moved D3 2.54 mm to (24.1, 19.1)
- moved JP1 2.54 mm to (20.3, 33.0)
- moved JP2 2.54 mm to (20.3, 27.9)
- moved R1 2.54 mm to (24.1, 14.6)
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Other:
- board text added: "Photon Battery Shield"
- board text removed: "Battery Shield for the Photon"
