File: Hardware/Photon Battery Shield.sch (EAGLE design)
At the start: 14 parts, among them J1 POWER_JACKSMD, U1 MCP73831, U2 MAX1704X

Commit message: Re-layed out, needs traces done
Parts:
- added D1, D2: MBRA140, SparkFun-DiscreteSemi:DIODE-SCHOTTKY-MBRA140
- added R5, R6: 10K, SparkFun-Resistors:10KOHM-1/10W-1%(0603)0603
- added SJ2: (no value), SparkFun-Passives:JUMPER-PAD-3-NC_BY_TRACE
- C1, C2: value 4.7uf -> 4.7uF; device SparkFun-Passives:CAP0402-CAP -> SparkFun-Passives:CAP0603-CAP
- C3: device SparkFun-Passives:CAP0402-CAP -> SparkFun-Passives:CAP0603-CAP
- JP3: value SPARK_PHOTON -> SPARK_PHOTONTEMPLATE; device template_temp:SPARK_PHOTON -> template_temp:SPARK_PHOTONTEMPLATE
- R1, R2, R3, R4: device SparkFun-Passives:RESISTOR0402-RES -> SparkFun-Passives:RESISTOR0603-RES
Connections:
- new net N$7: R5.2, SJ2.3
- new net N$8: D1.A, J1.PWR
- new net N$9: R6.2, SJ2.1
- net 3.3V: now also SJ2.2
- net SCL: now also R6.1
- net SDA: now also R5.1
- net VBAT: now also D2.A
- net VIN: now also D1.C, D2.C; no longer J1.PWR
Other:
- note removed: "SCL"
- note removed: "SDA"
- moved on the sheet: D11, J1, JP1, JP3, R1
